Commit message: updated geometry of mjcf to avoid meshes

File: assets/robot.urdf (robot description, URDF)
Before this commit: robot onshape, 7 links, 6 joints
Links:
- link right_foot: mass 0.1042736127887989861 -> 0.10427361278879899997
- link right_knee: mass 0.10414280809928128102 -> 0.1041428080992812949
- link thigh: mass 0.008228240608724240665 -> 0.0082282406087242354609
- link thigh_2: mass 0.008228240608724240665 -> 0.0082282406087242354609
Joints:
- joint left_foot: origin xyz=0.056830000071431546749 -0.00065000055707029567864 -0.059166631698607578815 rpy=-3.1415926535897926719 1.7837435507250453335e-16 -2.8163391732010532031 -> xyz=0.056830000071431546749 -0.00065000055707029220919 -0.059166631698607578815 rpy=-3.1415926535897926719 1.78374355072504558e-16 -2.8163391732010532031
- joint right_foot: origin xyz=0.056830000134848498994 0.00064999955300205913833 -0.05916663169859820437 rpy=-3.141592653589793116 6.4587986614972401477e-30 -0.51999566909108541068 -> xyz=0.056830000134848498994 0.00064999955300205566888 -0.05916663169859820437 rpy=-3.141592653589793116 6.4673233319424062448e-30 -0.51999566909108541068
- joint right_hip: origin xyz=0.021219150685801671519 0.082874409279697441866 0.095679164327205606932 rpy=-1.570796326794896336 7.1821472499178763301e-29 -3.4512664603419266487e-31 -> xyz=0.021219150685801671519 0.082874409279697441866 0.095679164327205606932 rpy=-1.570796326794896336 7.1821472499178763301e-29 -3.451266460341929714e-31
- joint right_knee: origin xyz=-0.032139381159561331014 0.038302222075878779306 -4.1633363423443370266e-17 rpy=3.141592653589793116 -4.9303806576313237838e-32 1.570796326794896558 -> xyz=-0.032139381159561331014 0.038302222075878779306 -4.1633363423443370266e-17 rpy=3.141592653589793116 -6.9333477998915039054e-32 1.570796326794896558

Commit message: Rerendered xml to realign root
xml should be close to final version. Should be trainable now.

File: assets/robot.urdf (robot description, URDF)
Before this commit: robot onshape, 7 links, 6 joints
Links:
- link left_foot: mass 0.10427362265243660111 -> 0.10427362265243658723
- link right_knee: mass 0.1041428080992812949 -> 0.10414280809928128102
- link thigh: mass 0.0082282406087242354609 -> 0.0082282406087242389303
- link thigh_2: mass 0.0082282406087242354609 -> 0.0082282406087242389303
Joints:
- joint left_foot: origin xyz=0.056830000071431546749 -0.00065000055707029220919 -0.059166631698607578815 rpy=-3.1415926535897926719 1.78374355072504558e-16 -2.8163391732010532031 -> xyz=0.056830000071432587583 -0.00065000055707035292452 -0.05916663169860798821 rpy=-3.1415926535897926719 1.78374355072504558e-16 -2.8163391732010532031
- joint left_hip: origin xyz=0.021219150623029883751 0.054074486336582044954 0.095579162487137395154 rpy=1.5707963267948970021 -2.2204460492503130808e-16 1.1241267899399416826e-29 -> xyz=-0.0050500014142475097012 -0.014401784459215430378 -0.079446995274444182078 rpy=1.5707963267948970021 -2.2204460492503130808e-16 1.1241267899399416826e-29
- joint left_knee: origin xyz=-0.032139381142254105916 -0.038302222060531534997 -6.2450045135165055399e-17 rpy=3.141592653589793116 -0 -1.570796326794896558 -> xyz=-0.032139381142254119794 -0.038302222060531507242 -5.7245874707234634116e-17 rpy=3.141592653589793116 -0 -1.570796326794896558
- joint right_foot: origin xyz=0.056830000134848498994 0.00064999955300205566888 -0.05916663169859820437 rpy=-3.141592653589793116 6.4673233319424062448e-30 -0.51999566909108541068 -> xyz=0.056830000134848485116 0.00064999955300212852727 -0.059166631698598218247 rpy=-3.141592653589793116 6.4673233319424062448e-30 -0.51999566909108541068
- joint right_hip: origin xyz=0.021219150685801671519 0.082874409279697441866 0.095679164327205606932 rpy=-1.570796326794896336 7.1821472499178763301e-29 -3.451266460341929714e-31 -> xyz=-0.0050500013514757358113 0.0143981384838995502 -0.079346993434376983378 rpy=-1.570796326794896336 7.1821472499178763301e-29 -3.451266460341929714e-31
- joint right_knee: origin xyz=-0.032139381159561331014 0.038302222075878779306 -4.1633363423443370266e-17 rpy=3.141592653589793116 -6.9333477998915039054e-32 1.570796326794896558 -> xyz=-0.032139381159561331014 0.038302222075878786245 -4.6837533851373791549e-17 rpy=3.141592653589793116 -6.9333477998915039054e-32 1.570796326794896558
